File: 24V-signal-to-5V.kicad_sch (KiCad schematic)
At the start: 5 parts, among them U3 4N35

Commit message: test archiving but using default lib
Parts:
- R5, R6, R7, R8: footprint project:R_Axial_DIN0207_L6.3mm_D2.5mm_P15.24mm_Horizontal -> Resistor_THT:R_Axial_DIN0207_L6.3mm_D2.5mm_P15.24mm_Horizontal; symbol archive:Device_R -> Device:R
- U3: footprint project:DIP-6_W7.62mm -> Package_DIP:DIP-6_W7.62mm; symbol archive:project_Isolator_4N35 -> Isolator:4N35
Changed lines of the file:
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@@
     (effects (font (size 1.27 1.27)) (justify left))
   )
-  (symbol (lib_id "archive:Device_R") (at 121.92 99.06 90) (mirror x)
+  (symbol (lib_id "Device:R") (at 121.92 99.06 90) (mirror x)
     (in_bom yes) (on_board yes)
     (property "Reference" "R5" (id 0) (at 123.19 96.52 90)
@@
       (effects (font (size 1.27 1.27)) (justify left))
     )
-    (property "Footprint" "project:R_Axial_DIN0207_L6.3mm_D2.5mm_P15.24mm_Horizontal" (id 2) (at 121.92 97.282 90)
+    (property "Footprint" "Resistor_THT:R_Axial_DIN0207_L6.3mm_D2.5mm_P15.24mm_Horizontal" (id 2) (at 121.92 97.282 90)
       (effects (font (size 1.27 1.27)) hide)
     )
@@
     (pin "2")
   )
-  (symbol (lib_id "archive:project_Isolator_4N35") (at 138.43 101.6 0)
+  (symbol (lib_id "Isolator:4N35") (at 138.43 101.6 0)
     (in_bom yes) (on_board yes)
     (property "Reference" "U3" (id 0) (at 138.43 109.6518 0))
     (property "Value" "4N35" (id 1) (at 138.43 107.3404 0))
-    (property "Footprint" "project:DIP-6_W7.62mm" (id 2) (at 133.35 106.68 0)
+    (property "Footprint" "Package_DIP:DIP-6_W7.62mm" (id 2) (at 133.35 106.68 0)
       (effects (font (size 1.27 1.27) italic) (justify left) hide)
     )
@@
     (pin "6")
   )
-  (symbol (lib_id "archive:Device_R") (at 165.1 101.6 270) (mirror x)
+  (symbol (lib_id "Device:R") (at 165.1 101.6 270) (mirror x)
     (in_bom yes) (on_board yes)
     (property "Reference" "R7" (id 0) (at 163.83 99.06 90)
@@
       (effects (font (size 1.27 1.27)) (justify left))
     )
-    (property "Footprint" "project:R_Axial_DIN0207_L6.3mm_D2.5mm_P15.24mm_Horizontal" (id 2) (at 165.1 103.378 90)
+    (property "Footprint" "Resistor_THT:R_Axial_DIN0207_L6.3mm_D2.5mm_P15.24mm_Horizontal" (id 2) (at 165.1 103.378 90)
       (effects (font (size 1.27 1.27)) hide)
     )
@@
     (pin "2")
   )
-  (symbol (lib_id "archive:Device_R") (at 165.1 91.44 270) (mirror x)
+  (symbol (lib_id "Device:R") (at 165.1 91.44 270) (mirror x)
     (in_bom yes) (on_board yes)
     (property "Reference" "R8" (id 0) (at 163.83 88.9 90)
@@
       (effects (font (size 1.27 1.27)) (justify left))
     )
-    (property "Footprint" "project:R_Axial_DIN0207_L6.3mm_D2.5mm_P15.24mm_Horizontal" (id 2) (at 165.1 93.218 90)
+    (property "Footprint" "Resistor_THT:R_Axial_DIN0207_L6.3mm_D2.5mm_P15.24mm_Horizontal" (id 2) (at 165.1 93.218 90)
       (effects (font (size 1.27 1.27)) hide)
     )
@@
     (pin "2")
   )
-  (symbol (lib_id "archive:Device_R") (at 165.1 110.49 270) (mirror x)
+  (symbol (lib_id "Device:R") (at 165.1 110.49 270) (mirror x)
     (in_bom yes) (on_board yes)
     (property "Reference" "R6" (id 0) (at 163.83 107.95 90)
@@
       (effects (font (size 1.27 1.27)) (justify left))
     )
-    (property "Footprint" "project:R_Axial_DIN0207_L6.3mm_D2.5mm_P15.24mm_Horizontal" (id 2) (at 165.1 112.268 90)
+    (property "Footprint" "Resistor_THT:R_Axial_DIN0207_L6.3mm_D2.5mm_P15.24mm_Horizontal" (id 2) (at 165.1 112.268 90)
       (effects (font (size 1.27 1.27)) hide)
     )
@@
     (pin "2")
   )
-  (symbol (lib_id "archive:power_+5V") (at 182.88 81.28 0) (mirror y)
+  (symbol (lib_id "power:+5V") (at 182.88 81.28 0) (mirror y)
     (in_bom yes) (on_board yes)
-    (property "Reference" "#PWR?" (id 0) (at 182.88 85.09 0)
+    (property "Reference" "#PWR0122" (id 0) (at 182.88 85.09 0)
       (effects (font (size 1.27 1.27)) hide)
     )
@@
     (pin "1")
   )
-  (symbol (lib_id "archive:power_GND") (at 128.27 106.68 0) (mirror y)
+  (symbol (lib_id "power:GND") (at 128.27 106.68 0) (mirror y)
     (in_bom yes) (on_board yes)
-    (property "Reference" "#PWR?" (id 0) (at 128.27 113.03 0)
+    (property "Reference" "#PWR0120" (id 0) (at 128.27 113.03 0)
       (effects (font (size 1.27 1.27)) hide)
     )
@@
     (pin "1")
   )
-  (symbol (lib_id "archive:power_GND") (at 176.53 121.92 0) (mirror y)
+  (symbol (lib_id "power:GND") (at 176.53 121.92 0) (mirror y)
     (in_bom yes) (on_board yes)
-    (property "Reference" "#PWR?" (id 0) (at 176.53 128.27 0)
+    (property "Reference" "#PWR0121" (id 0) (at 176.53 128.27 0)
       (effects (font (size 1.27 1.27)) hide)
     )

Commit message: components in place
Parts:
- R5, R6, R7, R8: footprint Resistor_THT:R_Axial_DIN0207_L6.3mm_D2.5mm_P15.24mm_Horizontal -> Resistor_SMD:R_0805_2012Metric_Pad1.20x1.40mm_HandSolder
Changed lines of the file:
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@@
       (effects (font (size 1.27 1.27)) (justify left))
     )
-    (property "Footprint" "Resistor_THT:R_Axial_DIN0207_L6.3mm_D2.5mm_P15.24mm_Horizontal" (id 2) (at 121.92 97.282 90)
+    (property "Footprint" "Resistor_SMD:R_0805_2012Metric_Pad1.20x1.40mm_HandSolder" (id 2) (at 121.92 97.282 90)
       (effects (font (size 1.27 1.27)) hide)
     )
@@
       (effects (font (size 1.27 1.27)) (justify left))
     )
-    (property "Footprint" "Resistor_THT:R_Axial_DIN0207_L6.3mm_D2.5mm_P15.24mm_Horizontal" (id 2) (at 165.1 103.378 90)
+    (property "Footprint" "Resistor_SMD:R_0805_2012Metric_Pad1.20x1.40mm_HandSolder" (id 2) (at 165.1 103.378 90)
       (effects (font (size 1.27 1.27)) hide)
     )
@@
       (effects (font (size 1.27 1.27)) (justify left))
     )
-    (property "Footprint" "Resistor_THT:R_Axial_DIN0207_L6.3mm_D2.5mm_P15.24mm_Horizontal" (id 2) (at 165.1 93.218 90)
+    (property "Footprint" "Resistor_SMD:R_0805_2012Metric_Pad1.20x1.40mm_HandSolder" (id 2) (at 165.1 93.218 90)
       (effects (font (size 1.27 1.27)) hide)
     )
@@
       (effects (font (size 1.27 1.27)) (justify left))
     )
-    (property "Footprint" "Resistor_THT:R_Axial_DIN0207_L6.3mm_D2.5mm_P15.24mm_Horizontal" (id 2) (at 165.1 112.268 90)
+    (property "Footprint" "Resistor_SMD:R_0805_2012Metric_Pad1.20x1.40mm_HandSolder" (id 2) (at 165.1 112.268 90)
       (effects (font (size 1.27 1.27)) hide)
     )
