File: extruder_controll.kicad_sch (KiCad schematic)
At the start: 15 parts, among them J1 Conn_01x04_Male, J3 Conn_01x06_Male, M1 Stepper_Motor_bipolar, P1 Power, P2 Analog, P3 Digital, P4 Digital, P5 CONN_01X01, P6 CONN_01X01, P7 CONN_01X01, P8 CONN_01X01, U1 MotionKing_2L415B

Commit message: test archiving but using default lib
Parts:
- C1, C2: footprint project:CP_Radial_D6.3mm_P2.50mm -> Capacitor_THT:CP_Radial_D6.3mm_P2.50mm; symbol archive:Device_CP -> Device:C_Polarized
- J1: footprint project:Molex_Micro-Fit_3.0_43045-0400_2x02_P3.00mm_Horizontal -> Connector_Molex:Molex_Micro-Fit_3.0_43045-0400_2x02_P3.00mm_Horizontal; symbol archive:project_Connector_Conn_01x04_Male -> Connector_Generic:Conn_01x04
- J3: footprint project:Molex_Micro-Fit_3.0_43045-0600_2x03_P3.00mm_Horizontal -> Connector_Molex:Molex_Micro-Fit_3.0_43045-0600_2x03_P3.00mm_Horizontal; symbol archive:project_Connector_Conn_01x06_Male -> Connector_Generic:Conn_01x06
- M1: symbol archive:project_Motor_Stepper_Motor_bipolar -> Motor:Stepper_Motor_bipolar
- P1, P4: footprint Socket_Arduino_Uno:Socket_Strip_Arduino_1x08 -> project:Socket_Strip_Arduino_1x08; symbol archive:Connector_Generic_Conn_01x08 -> Connector_Generic:Conn_01x08
- P2: footprint Socket_Arduino_Uno:Socket_Strip_Arduino_1x06 -> project:Socket_Strip_Arduino_1x06; symbol archive:Connector_Generic_Conn_01x06 -> Connector_Generic:Conn_01x06
- P3: footprint Socket_Arduino_Uno:Socket_Strip_Arduino_1x10 -> project:Socket_Strip_Arduino_1x10; symbol archive:Connector_Generic_Conn_01x10 -> Connector_Generic:Conn_01x10
- P5, P6, P7, P8: footprint Socket_Arduino_Uno:Arduino_1pin -> project:Arduino_1pin; symbol archive:Connector_Generic_Conn_01x01 -> Connector_Generic:Conn_01x01
- PS1: symbol archive:project_R-78B5.0-1.0 -> project:project_R-78B5.0-1.0
- U1: symbol archive:project_MotionKing_2L415B -> project:project_MotionKing_2L415B

Commit message: components in place
Parts:
- removed PS1: R-78B5.0-1.0, project:R-78B5.0-1.0, symbol project:project_R-78B5.0-1.0
- added J2: USB_C_Receptacle, project:MOLEX_105450-0101, symbol Connector:USB_C_Receptacle
- added U4: JTD2024S05, Converter_DCDC:Converter_DCDC_XP_POWER_JTDxxxxxxx_THT, symbol Converter_DCDC:JTD2024S05
Connections:
- net +24V: now also U4.1 (+VIN)
- net +5V: now also J2.A4 (VBUS), J2.A9 (VBUS), J2.B4 (VBUS), J2.B9 (VBUS), U4.5 (-VOUT)
- net 0V: now also J2.A1 (GND), J2.A12 (GND), J2.B1 (GND), J2.B12 (GND), U4.3 (+VOUT)
- no-connect marks 41 -> 58
Other:
- moved on the sheet: C1
