File: 24V_plc_integration_shield/extruder_controll-backups/extruder_controll-2022-01-13_191503/24V-signal-to-5V.kicad_sch (KiCad schematic)
At the start: 5 parts, among them U3 4N35

Commit message: big commit after big mistake
Parts:
- added D3: LED, LED_THT:LED_D5.0mm, symbol Device:LED
- added R11: 150 Ω, Resistor_THT:R_Axial_DIN0207_L6.3mm_D2.5mm_P2.54mm_Vertical, symbol Device:R
- R5, R7, R8: footprint Resistor_SMD:R_0805_2012Metric_Pad1.20x1.40mm_HandSolder -> Resistor_THT:R_Axial_DIN0207_L6.3mm_D2.5mm_P2.54mm_Vertical
- R6: value 4.7 k Ω -> 4.7 kΩ; footprint Resistor_SMD:R_0805_2012Metric_Pad1.20x1.40mm_HandSolder -> Resistor_THT:R_Axial_DIN0207_L6.3mm_D2.5mm_P2.54mm_Vertical
- U3: footprint Package_DIP:DIP-6_W7.62mm -> Package_DIP:DIP-6_W7.62mm_Socket
Connections:
- net 5V-signal: now also D3.2 (A)
- net GND: now also R11.1
- new net: D3.1 (K), R11.2
Changed lines of the file:
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@@
     (title "EXTRUDER CONTROL")
     (date "2021-11-01")
+    (rev "v2")
     (company "bioDigital Matter Lab")
     (comment 1 "Anton Tetov")
   )
-  (junction (at 176.53 110.49) (diameter 0) (color 0 0 0 0)
-  )
   (junction (at 149.86 110.49) (diameter 0) (color 0 0 0 0)
   )
+  (junction (at 149.86 118.11) (diameter 0) (color 0 0 0 0)
+  )
+  (junction (at 180.34 128.27) (diameter 0) (color 0 0 0 0)
+  )
+  (junction (at 180.34 110.49) (diameter 0) (color 0 0 0 0)
+  )
   (wire (pts (xy 146.05 99.06) (xy 149.86 99.06))
     (stroke (width 0) (type default) (color 0 0 0 0))
@@
     (stroke (width 0) (type default) (color 0 0 0 0))
   )
+  (wire (pts (xy 168.91 110.49) (xy 180.34 110.49))
+    (stroke (width 0) (type default) (color 0 0 0 0))
+  )
   (wire (pts (xy 149.86 91.44) (xy 161.29 91.44))
     (stroke (width 0) (type default) (color 0 0 0 0))
@@
     (stroke (width 0) (type default) (color 0 0 0 0))
   )
-  (wire (pts (xy 176.53 110.49) (xy 176.53 91.44))
-    (stroke (width 0) (type default) (color 0 0 0 0))
-  )
-  (wire (pts (xy 168.91 91.44) (xy 176.53 91.44))
+  (wire (pts (xy 149.86 118.11) (xy 149.86 128.27))
+    (stroke (width 0) (type default) (color 0 0 0 0))
+  )
+  (wire (pts (xy 180.34 110.49) (xy 180.34 91.44))
+    (stroke (width 0) (type default) (color 0 0 0 0))
+  )
+  (wire (pts (xy 168.91 91.44) (xy 180.34 91.44))
     (stroke (width 0) (type default) (color 0 0 0 0))
   )
@@
     (stroke (width 0) (type default) (color 0 0 0 0))
   )
-  (wire (pts (xy 182.88 101.6) (xy 182.88 81.28))
+  (wire (pts (xy 175.26 101.6) (xy 175.26 81.28))
+    (stroke (width 0) (type default) (color 0 0 0 0))
+  )
+  (wire (pts (xy 173.99 128.27) (xy 180.34 128.27))
     (stroke (width 0) (type default) (color 0 0 0 0))
   )
@@
     (stroke (width 0) (type default) (color 0 0 0 0))
   )
-  (wire (pts (xy 176.53 110.49) (xy 176.53 121.92))
+  (wire (pts (xy 180.34 110.49) (xy 180.34 128.27))
+    (stroke (width 0) (type default) (color 0 0 0 0))
+  )
+  (wire (pts (xy 180.34 128.27) (xy 180.34 135.89))
     (stroke (width 0) (type default) (color 0 0 0 0))
   )
@@
     (stroke (width 0) (type default) (color 0 0 0 0))
   )
-  (wire (pts (xy 168.91 101.6) (xy 182.88 101.6))
+  (wire (pts (xy 168.91 101.6) (xy 175.26 101.6))
+    (stroke (width 0) (type default) (color 0 0 0 0))
+  )
+  (wire (pts (xy 161.29 128.27) (xy 166.37 128.27))
+    (stroke (width 0) (type default) (color 0 0 0 0))
+  )
+  (wire (pts (xy 149.86 128.27) (xy 153.67 128.27))
     (stroke (width 0) (type default) (color 0 0 0 0))
   )
   (wire (pts (xy 146.05 104.14) (xy 149.86 104.14))
-    (stroke (width 0) (type default) (color 0 0 0 0))
-  )
-  (wire (pts (xy 176.53 110.49) (xy 168.91 110.49))
     (stroke (width 0) (type default) (color 0 0 0 0))
   )
@@
       (effects (font (size 1.27 1.27)) (justify left))
     )
-    (property "Footprint" "Resistor_SMD:R_0805_2012Metric_Pad1.20x1.40mm_HandSolder" (id 2) (at 121.92 97.282 90)
+    (property "Footprint" "Resistor_THT:R_Axial_DIN0207_L6.3mm_D2.5mm_P2.54mm_Vertical" (id 2) (at 121.92 97.282 90)
       (effects (font (size 1.27 1.27)) hide)
     )
@@
     (property "Reference" "U3" (id 0) (at 138.43 109.6518 0))
     (property "Value" "4N35" (id 1) (at 138.43 107.3404 0))
-    (property "Footprint" "Package_DIP:DIP-6_W7.62mm" (id 2) (at 133.35 106.68 0)
+    (property "Footprint" "Package_DIP:DIP-6_W7.62mm_Socket" (id 2) (at 133.35 106.68 0)
       (effects (font (size 1.27 1.27) italic) (justify left) hide)
     )
@@
       (effects (font (size 1.27 1.27)) (justify left))
     )
-    (property "Footprint" "Resistor_SMD:R_0805_2012Metric_Pad1.20x1.40mm_HandSolder" (id 2) (at 165.1 103.378 90)
+    (property "Footprint" "Resistor_THT:R_Axial_DIN0207_L6.3mm_D2.5mm_P2.54mm_Vertical" (id 2) (at 165.1 103.378 90)
       (effects (font (size 1.27 1.27)) hide)
     )
@@
       (effects (font (size 1.27 1.27)) (justify left))
     )
-    (property "Footprint" "Resistor_SMD:R_0805_2012Metric_Pad1.20x1.40mm_HandSolder" (id 2) (at 165.1 93.218 90)
+    (property "Footprint" "Resistor_THT:R_Axial_DIN0207_L6.3mm_D2.5mm_P2.54mm_Vertical" (id 2) (at 165.1 93.218 90)
       (effects (font (size 1.27 1.27)) hide)
     )
@@
       (effects (font (size 1.27 1.27)) (justify left))
     )
-    (property "Value" "4.7 k Ω" (id 1) (at 161.29 113.03 90)
-      (effects (font (size 1.27 1.27)) (justify left))
-    )
-    (property "Footprint" "Resistor_SMD:R_0805_2012Metric_Pad1.20x1.40mm_HandSolder" (id 2) (at 165.1 112.268 90)
+    (property "Value" "4.7 kΩ" (id 1) (at 161.29 113.03 90)
+      (effects (font (size 1.27 1.27)) (justify left))
+    )
+    (property "Footprint" "Resistor_THT:R_Axial_DIN0207_L6.3mm_D2.5mm_P2.54mm_Vertical" (id 2) (at 165.1 112.268 90)
       (effects (font (size 1.27 1.27)) hide)
     )
@@
     (pin "2")
   )
-  (symbol (lib_id "power:+5V") (at 182.88 81.28 0) (mirror y)
-    (in_bom yes) (on_board yes)
-    (property "Reference" "#PWR0122" (id 0) (at 182.88 85.09 0)
-      (effects (font (size 1.27 1.27)) hide)
-    )
-    (property "Value" "+5V" (id 1) (at 182.499 76.8858 0))
-    (property "Footprint" "" (id 2) (at 182.88 81.28 0)
-      (effects (font (size 1.27 1.27)) hide)
-    )
-    (property "Datasheet" "" (id 3) (at 182.88 81.28 0)
+  (symbol (lib_id "power:+5V") (at 175.26 81.28 0) (mirror y)
+    (in_bom yes) (on_board yes)
+    (property "Reference" "#PWR0122" (id 0) (at 175.26 85.09 0)
+      (effects (font (size 1.27 1.27)) hide)
+    )
+    (property "Value" "+5V" (id 1) (at 174.879 76.8858 0))
+    (property "Footprint" "" (id 2) (at 175.26 81.28 0)
+      (effects (font (size 1.27 1.27)) hide)
+    )
+    (property "Datasheet" "" (id 3) (at 175.26 81.28 0)
       (effects (font (size 1.27 1.27)) hide)
     )
@@
     (pin "1")
   )
-  (symbol (lib_id "power:GND") (at 176.53 121.92 0) (mirror y)
-    (in_bom yes) (on_board yes)
-    (property "Reference" "#PWR0121" (id 0) (at 176.53 128.27 0)
-      (effects (font (size 1.27 1.27)) hide)
-    )
-    (property "Value" "GND" (id 1) (at 176.403 126.3142 0))
-    (property "Footprint" "" (id 2) (at 176.53 121.92 0)
-      (effects (font (size 1.27 1.27)) hide)
-    )
-    (property "Datasheet" "" (id 3) (at 176.53 121.92 0)
-      (effects (font (size 1.27 1.27)) hide)
-    )
-    (pin "1")
+  (symbol (lib_id "power:GND") (at 180.34 135.89 0) (mirror y)
+    (in_bom yes) (on_board yes)
+    (property "Reference" "#PWR0121" (id 0) (at 180.34 142.24 0)
+      (effects (font (size 1.27 1.27)) hide)
+    )
+    (property "Value" "GND" (id 1) (at 180.213 140.2842 0))
+    (property "Footprint" "" (id 2) (at 180.34 135.89 0)
+      (effects (font (size 1.27 1.27)) hide)
+    )
+    (property "Datasheet" "" (id 3) (at 180.34 135.89 0)
+      (effects (font (size 1.27 1.27)) hide)
+    )
+    (pin "1")
+  )
+  (symbol (lib_id "Device:R") (at 170.18 128.27 270) (mirror x)
+    (in_bom yes) (on_board yes)
+    (property "Reference" "R11" (id 0) (at 168.91 125.73 90)
+      (effects (font (size 1.27 1.27)) (justify left))
+    )
+    (property "Value" "150 Ω" (id 1) (at 166.37 130.81 90)
+      (effects (font (size 1.27 1.27)) (justify left))
+    )
+    (property "Footprint" "Resistor_THT:R_Axial_DIN0207_L6.3mm_D2.5mm_P2.54mm_Vertical" (id 2) (at 170.18 130.048 90)
+      (effects (font (size 1.27 1.27)) hide)
+    )
+    (property "Datasheet" "~" (id 3) (at 170.18 128.27 0)
+      (effects (font (size 1.27 1.27)) hide)
+    )
+    (pin "1")
+    (pin "2")
+  )
+  (symbol (lib_id "Device:LED") (at 157.48 128.27 180)
+    (in_bom yes) (on_board yes) (fields_autoplaced)
+    (property "Reference" "D3" (id 0) (at 159.0675 120.65 0))
+    (property "Value" "LED" (id 1) (at 159.0675 123.19 0))
+    (property "Footprint" "LED_THT:LED_D5.0mm" (id 2) (at 157.48 128.27 0)
+      (effects (font (size 1.27 1.27)) hide)
+    )
+    (property "Datasheet" "~" (id 3) (at 157.48 128.27 0)
+      (effects (font (size 1.27 1.27)) hide)
+    )
+    (pin "1")
+    (pin "2")
   )
 )
